Commit message: arm_test and color

File: urdf/car.urdf.xacro (robot description, xacro)
@@ -939,4 +939,5 @@
       velocity="0" />
   </joint>
+<!-- Controllers -->
 <ros2_control name="GazeboSystem" type="system">
  <hardware>
@@ -1095,12 +1096,14 @@
     </plugin>
  </gazebo>
- <xacro:macro name="body_color">
-    <visual>
-    <material>
-        <ambient>0.8 0.558823529411765 0.1 1</ambient>
-        <diffuse>0.8 0.558823529411765 0.1 1</diffuse>
-        <specular>0.1 0.1 0.1 1</specular>
-        <emissive>0 0 0 0</emissive>
-    </material>
+<!-- Controllers -->
+<!-- color -->
+<xacro:macro name="body_color">
+    <visual>
+        <material>
+            <ambient>0.1 0.1 0.8 1</ambient> <!-- Dark Blue -->
+            <diffuse>0.1 0.1 0.8 1</diffuse> <!-- Dark Blue -->
+            <specular>0.1 0.1 0.1 1</specular>
+            <emissive>0 0 0 0</emissive>
+        </material>
     </visual>
 </xacro:macro>
@@ -1121,3 +1124,101 @@
     <xacro:lidar_color />
 </gazebo>
+<xacro:macro name="hinge_color">
+    <visual>
+        <material>
+           <ambient>0.8 0 0 1</ambient> <!-- Bright Red -->
+            <diffuse>0.8 0 0 1</diffuse> <!-- Bright Red -->
+            <specular>0.1 0.1 0.1 1</specular>
+            <emissive>0 0 0 0</emissive>
+        </material>
+    </visual>
+</xacro:macro>
+<gazebo reference="left_hinge_back">
+    <xacro:hinge_color />
+</gazebo>
+<gazebo reference="left_hinge_front">
+    <xacro:hinge_color />
+</gazebo>
+<gazebo reference="right_hinge_back">
+    <xacro:hinge_color />
+</gazebo>
+<gazebo reference="right_hinge_front">
+    <xacro:hinge_color />
+</gazebo>
+<xacro:macro name="tires">
+    <visual>
+        <material>
+            <ambient>0.3 0.3 0.3 1</ambient> <!-- Dark Gray -->
+            <diffuse>0.3 0.3 0.3 1</diffuse> <!-- Dark Gray -->
+            <specular>0.1 0.1 0.1 1</specular>
+            <emissive>0 0 0 0</emissive>
+        </material>
+    </visual>
+</xacro:macro>
+<gazebo reference="Left_wheel_front">
+    <xacro:tires />
+</gazebo>
+<gazebo reference="right_wheel_back">
+    <xacro:tires />
+</gazebo>
+<gazebo reference="left_wheel_back">
+    <xacro:tires />
+</gazebo>
+<gazebo reference="right_wheel_front">
+    <xacro:tires />
+</gazebo>
+<gazebo reference="arm_base">
+    <xacro:hinge_color />
+</gazebo>
+<xacro:macro name="ur5">
+    <visual>
+        <material>
+            <ambient>0.529 0.808 0.922 1</ambient> <!-- Light Blue -->
+            <diffuse>0.529 0.808 0.922 1</diffuse> <!-- Light Blue -->
+            <specular>0.1 0.1 0.1 1</specular>
+            <emissive>0 0 0 0</emissive>
+        </material>
+    </visual>
+</xacro:macro>
+<gazebo reference="link_1">
+    <xacro:ur5 />
+</gazebo>
+<gazebo reference="link_2">
+    <xacro:ur5 />
+</gazebo>
+<gazebo reference="link_3">
+    <xacro:ur5 />
+</gazebo>
+<gazebo reference="link_4">
+    <xacro:ur5 />
+</gazebo>
+<gazebo reference="link_5">
+    <xacro:ur5 />
+</gazebo>
+<gazebo reference="link_6">
+    <xacro:ur5 />
+</gazebo>
+<!-- color -->
+<!-- plugins -->
+<!-- vacuum gripper -->
+<gazebo>
+  <plugin name='vacuum_gripper' filename='libgazebo_ros_vacuum_gripper.so'>
+    <!-- This part can be commented out if not required -->
+    <ros>
+      <!-- Add a namespace -->
+      <namespace>/demo</namespace>
+      <!-- Remapping service and topic names -->
+      <remapping>switch:=custom_switch</remapping>
+      <remapping>grasping:=custom_grasping</remapping>
+    </ros>
+    <!-- Link associated with gripper -->
+    <link_name>link_6</link_name>
+    <!-- Max distance to attract entities -->
+    <max_distance>10.0</max_distance>
+    <!-- List of entities to be not attracted by the gripper -->
+    <fixed>ground_plane</fixed>
+    <fixed>wall</fixed>
+  </plugin>
+</gazebo>
+<!-- plugins -->
 </robot>

Commit message: IKsolver written

File: urdf/car.urdf.xacro (robot description, xacro)
@@ -485,5 +485,5 @@
       xyz="0 0 -1" />
   </joint>
-  <link
+  <!-- <link
     name="lidar_link">
     <inertial>
@@ -537,5 +537,5 @@
     <axis
       xyz="0 0 0" />
-  </joint>
+  </joint> -->
   <link
     name="arm_base">
@@ -1111,5 +1111,5 @@
     <xacro:body_color />
 </gazebo>
-<xacro:macro name="lidar_color">
+<!-- <xacro:macro name="lidar_color">
     <visual>
         <material>
@@ -1123,5 +1123,5 @@
 <gazebo reference="lidar_link">
     <xacro:lidar_color />
-</gazebo>
+</gazebo> -->
 <xacro:macro name="hinge_color">
     <visual>

Commit message: updated files

File: urdf/car.urdf.xacro (robot description, xacro)
@@ -636,5 +636,5 @@
     <origin
       xyz="0 0 0.087"
-      rpy="0 0 3.1416" />
+      rpy="0 0 0" />
     <parent
       link="arm_base" />
@@ -644,6 +644,6 @@
       xyz="0 0 -1" />
     <limit
-      lower="-3.14"
-      upper="3.14"
+      lower="-6.28"
+      upper="6.28"
       effort="0"
       velocity="0" />
@@ -694,5 +694,5 @@
     <origin
       xyz="7.1962E-05 0.135 0"
-      rpy="-1.5708 0.010572 -0.00053305" />
+      rpy="-1.5708 1.5708 -0.00053305" />
     <parent
       link="link_1" />
@@ -702,6 +702,6 @@
       xyz="0 0 -1" />
     <limit
-      lower="-3.14"
-      upper="3.14"
+      lower="-6.28"
+      upper="6.28"
       effort="0"
       velocity="0" />
@@ -752,5 +752,5 @@
     <origin
       xyz="0 -0.425 -0.11995"
-      rpy="3.1416 0 -3.1319" />
+      rpy="3.1416 0 1.57079" />
     <parent
       link="link_2" />
@@ -760,6 +760,6 @@
       xyz="0 0 1" />
     <limit
-      lower="-3.14"
-      upper="3.14"
+      lower="-6.28"
+      upper="6.28"
       effort="0"
       velocity="0" />
@@ -810,5 +810,5 @@
     <origin
       xyz="-0.39225 0 -0.09492"
-      rpy="3.1416 0 0.52654" />
+      rpy="3.1416 0 0" />
     <parent
       link="link_3" />
@@ -818,6 +818,6 @@
       xyz="0 0 1" />
     <limit
-      lower="-3.14"
-      upper="3.14"
+      lower="-6.28"
+      upper="6.28"
       effort="0"
       velocity="0" />
@@ -868,5 +868,5 @@
     <origin
       xyz="0 -0.09492 0"
-      rpy="-1.5708 -1.4334 3.1416" />
+      rpy="-1.5708 0 3.1416" />
     <parent
       link="link_4" />
@@ -876,6 +876,6 @@
       xyz="0 0 1" />
     <limit
-      lower="-3.14"
-      upper="3.14"
+      lower="-6.28"
+      upper="6.28"
       effort="0"
       velocity="0" />
@@ -934,6 +934,6 @@
       xyz="0 0 1" />
     <limit
-      lower="-3.14"
-      upper="3.14"
+      lower="-6.28"
+      upper="6.28"
       effort="0"
       velocity="0" />
@@ -1044,6 +1044,6 @@
  <joint name="link_joint_1">
      <command_interface name="position">
-         <param name="min">-3.14</param>
-         <param name="max">3.14</param>
+         <param name="min">-6.28</param>
+         <param name="max">6.28</param>
      </command_interface>
      <state_interface name="position"/>
@@ -1202,4 +1202,27 @@
 <!-- plugins -->
 <!-- vacuum gripper -->
+<link name="vacuum_effector">
+    <gravity>0</gravity>
+    <visual>
+      <origin rpy="0 0 0" xyz="0 0 0"/>
+      <geometry>
+        <box size="0.05 0.02 0.05"/>
+      </geometry>
+      <material name="transparent">
+        <color rgba="0 0 0 0"/>
+      </material>
+    </visual>
+    <inertial>
+      <origin rpy="0 0 0" xyz="0.000000 0.000000 0.000000"/>
+      <mass value="0.0001"/>
+      <inertia ixx="1e-08" ixy="0" ixz="0" iyy="1e-08" iyz="0" izz="1e-08"/>
+    </inertial>
+  </link>
+  <joint name="end_effector" type="revolute">
+    <parent link="link_6" />
+    <child link="vacuum_effector" />
+    <origin rpy="1.5708 0 0" xyz="0 0 0.01" />
+    <limit effort="30" velocity="1.0" lower="0" upper="0" />
+  </joint>
 <gazebo>
   <plugin name='vacuum_gripper' filename='libgazebo_ros_vacuum_gripper.so'>
@@ -1213,5 +1236,5 @@
     </ros>
     <!-- Link associated with gripper -->
-    <link_name>link_6</link_name>
+    <link_name>vacuum_effector</link_name>
     <!-- Max distance to attract entities -->
     <max_distance>10.0</max_distance>
